Commit message: implementation

File: lidar_calibration/urdf/hector_multisensor_head_with_error.urdf (robot description, URDF)
Before this commit: robot hector_multisensor_head, 10 links, 9 joints
Joints:
- joint head_link_hokuyo_laser_joint: origin xyz=0.005 0.005 0 rpy=0.1 0.1 0.1 -> xyz=0 0 0 rpy=0 0.1 0

Commit message: added ceres solver

File: lidar_calibration/urdf/hector_multisensor_head_with_error.urdf (robot description, URDF)
Before this commit: robot hector_multisensor_head, 10 links, 9 joints
Joints:
- joint head_link_hokuyo_laser_joint: origin xyz=0 0 0 rpy=0 0.1 0 -> xyz=0 0.01 0 rpy=0 0 0

Commit message: Filter invalid points after mls, removed unused files, calibration now running

File: lidar_calibration/urdf/hector_multisensor_head_with_error.urdf (robot description, URDF)
Before this commit: robot hector_multisensor_head, 10 links, 9 joints
Joints:
- joint head_link_hokuyo_laser_joint: origin xyz=0 0.01 0 rpy=0 0 0 -> xyz=0 0 0 rpy=0 0 0

Commit message: debug publishing and box filter for points that are too close

File: lidar_calibration/urdf/hector_multisensor_head_with_error.urdf (robot description, URDF)
Before this commit: robot hector_multisensor_head, 10 links, 9 joints
Joints:
- joint head_link_hokuyo_laser_joint: origin xyz=0 0 0 rpy=0 0 0 -> xyz=0 0.05 0.05 rpy=0 0 0

Commit message: started reworking for different error function

File: lidar_calibration/urdf/hector_multisensor_head_with_error.urdf (robot description, URDF)
Before this commit: robot hector_multisensor_head, 10 links, 9 joints
Joints:
- joint head_link_hokuyo_laser_joint: origin xyz=0 0.05 0.05 rpy=0 0 0 -> xyz=0 -0.05 -0.05 rpy=0 0 0

Commit message: calibration in first working state

File: lidar_calibration/urdf/hector_multisensor_head_with_error.urdf (robot description, URDF)
Before this commit: robot hector_multisensor_head, 10 links, 9 joints
Joints:
- joint head_link_hokuyo_laser_joint: origin xyz=0 -0.05 -0.05 rpy=0 0 0 -> xyz=0 0.05 0.05 rpy=0 0 0.1

Commit message: added ground plane detection for roll offset

File: lidar_calibration/urdf/hector_multisensor_head_with_error.urdf (robot description, URDF)
Before this commit: robot hector_multisensor_head, 10 links, 9 joints
Joints:
- joint head_link_hokuyo_laser_joint: origin xyz=0 0.05 0.05 rpy=0 0 0.1 -> xyz=0 0.05 0 rpy=0.1 0 0

Commit message: calibration can now be saved to disk. added option to specify different laser frame orientation

File: lidar_calibration/urdf/hector_multisensor_head_with_error.urdf (robot description, URDF)
Before this commit: robot hector_multisensor_head, 10 links, 9 joints
Joints:
- joint head_lidar_spinning_joint: origin xyz=0.061 0.0 0.134 rpy=0 0 0 -> xyz=0.061 0 0.134 rpy=0 0 0
- joint head_link_hokuyo_laser_joint: origin xyz=0 0.05 0 rpy=0.1 0 0 -> xyz=0 0.05 0.05 rpy=0 0 0

Commit message: transforms now retrieved at calibration start. fixed bug with negative roll angles. refactoring

File: lidar_calibration/urdf/hector_multisensor_head_with_error.urdf (robot description, URDF)
Before this commit: robot hector_multisensor_head, 10 links, 9 joints
Joints:
- joint head_link_hokuyo_laser_joint: origin xyz=0 0.05 0.05 rpy=0 0 0 -> xyz=0.0 0 0 rpy=-0.1 0 0

Commit message: fixed bug when roll of ground detecting was applied

File: lidar_calibration/urdf/hector_multisensor_head_with_error.urdf (robot description, URDF)
Before this commit: robot hector_multisensor_head, 10 links, 9 joints
Joints:
- joint head_link_hokuyo_laser_joint: origin xyz=0.0 0 0 rpy=-0.1 0 0 -> xyz=0.0 0.05 0.05 rpy=0.2 0.2 0.2

Commit message: changed dependencies, so ceres no longer needs to be built from source

File: lidar_calibration/urdf/hector_multisensor_head_with_error.urdf (robot description, URDF)
Before this commit: robot hector_multisensor_head, 10 links, 9 joints
Links:
- link head_link_hokuyo_laser_frame: mass 0.270 -> 0.070
Joints:
- joint head_link_hokuyo_laser_joint: origin xyz=0.0 0.05 0.05 rpy=0.2 0.2 0.2 -> xyz=0.0 0.05 0.05 rpy=0.1 0.1 0.1

Commit message: multi lidar calibration - initial commit

File: lidar_calibration/urdf/hector_multisensor_head_with_error.urdf (robot description, URDF)
Before this commit: robot hector_multisensor_head, 10 links, 9 joints
Joints:
- joint head_link_hokuyo_laser_joint: origin xyz=0.0 0.05 0.05 rpy=0.1 0.1 0.1 -> xyz=0.0 0.0 0.0 rpy=-0.4 0 0

Commit message: replaced functions in lidar_calibration with lib functions

File: lidar_calibration/urdf/hector_multisensor_head_with_error.urdf (robot description, URDF)
Before this commit: robot hector_multisensor_head, 10 links, 9 joints
Joints:
- joint head_link_hokuyo_laser_joint: origin xyz=0.0 0.0 0.0 rpy=-0.4 0 0 -> xyz=0.0 -0.05 0.05 rpy=0 0.1 -0.1
