Commit message: launch file updates to evaluation

File: lidar_calibration/urdf/hector_multisensor_head_with_error_new.urdf (robot description, URDF)
Before this commit: robot hector_multisensor_head, 10 links, 9 joints
Links:
- removed link head_cam_depth_frame
- removed link head_cam_depth_optical_frame
- removed link head_cam_rgb_frame
- removed link head_cam_rgb_optical_frame
- link head_cam_link: geometry collision box size=0.007 0.130 0.02; visual box size=0.007 0.130 0.02
- link head_link: mass 0.1 -> 0.8
- link head_link_hokuyo_laser_frame: mass 0.070 -> 0.270; geometry collision cylinder length=0.079 radius=0.0735; visual mesh filename=package://hector_sensors_description/meshes/hokuyo_utm30lx/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
Joints:
- removed joint head_cam_depth_joint
- removed joint head_cam_depth_optical_joint
- removed joint head_cam_rgb_joint
- removed joint head_cam_rgb_optical_joint
- joint head_cam_joint: origin xyz=0.0385 0.0 0.2385 rpy=0 0 0 -> xyz=0.015 -0.05 0.181 rpy=0 0.261799 0
- joint head_lidar_spinning_joint: origin xyz=0.061 0 0.134 rpy=0 0 0 -> xyz=0.061 0.0 0.083 rpy=0 0 0
- joint head_link_hokuyo_laser_joint: origin xyz=0 0 0 rpy=0 0 0 -> xyz=0 0.05 0.05 rpy=0 0.1 0.1

File: multi_lidar_calibration/urdf/realsense_error.urdf (robot description, URDF)
Before this commit: robot hector_multisensor_head, 10 links, 9 joints
Links:
- removed link head_cam_depth_frame
- removed link head_cam_depth_optical_frame
- removed link head_cam_rgb_frame
- removed link head_cam_rgb_optical_frame
- link base: geometry 
- link head_cam_link: geometry collision box size=0.007 0.130 0.02; visual box size=0.007 0.130 0.02
- link head_link: mass 0.1 -> 0.8
- link head_link_hokuyo_laser_frame: mass 0.070 -> 0.270; geometry collision cylinder length=0.079 radius=0.0735; visual mesh filename=package://hector_sensors_description/meshes/hokuyo_utm30lx/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
Joints:
- removed joint head_cam_depth_joint
- removed joint head_cam_depth_optical_joint
- removed joint head_cam_rgb_joint
- removed joint head_cam_rgb_optical_joint
- joint fixed1: origin xyz=0.0 0.0 0.5 rpy=0 0 0 -> xyz=0.0 0.0 0.1 rpy=0 0 0
- joint fixed2: origin xyz=0.0 0.0 0.5 rpy=0 0 0 -> xyz=0.0 0.0 0.1 rpy=0 0 0
- joint head_cam_joint: origin xyz=0.0385 0.0 0.2385 rpy=0 0 0 -> xyz=0.065 0 0.231 rpy=0.1 0.1 0.1
- joint head_lidar_spinning_joint: origin xyz=0.061 0 0.134 rpy=0 0 0 -> xyz=0.061 0.0 0.083 rpy=0 0 0
