Commit message: fixed accumulation of iterative calibration results

File: multi_lidar_calibration/urdf/realsense_error.urdf (robot description, URDF)
Before this commit: robot hector_multisensor_head, 6 links, 5 joints
Joints:
- joint head_cam_joint: origin xyz=0.065 0 0.231 rpy=0.1 0.1 0.1 -> xyz=0.035 -0.03 0.201 rpy=0.05 0.05 0.05
